File: hardware/energy_monitor/energy_monitor.kicad_pcb (KiCad board)
At the start: 4 copper layers, 102.8 x 86.9 mm, 145 parts, among them J1 Screw_Terminal_01x03, J2 Screw_Terminal_01x04, J3 Screw_Terminal_01x04, J4 Screw_Terminal_01x04, J5 USB_OTG, Q1 MMBT2222, Q2 MMBT2222, U1 RAC04, U2 TPS730, U3 TPS723, U4 ADS131E08, U5 AP2112, U6 CP2104, U7 ESP-WROOM-32U, U8 ISO7421, U9 ISO7420

Commit message: Minor PCB tweaks and created gerbers
Routing:
- net /RESET: track 47.1 -> 43.7 mm
- net Net-(R13-Pad1): track 11.6 -> 10.8 mm
Changed lines of the file:
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@@
     (thickness 1.6)
     (drawings 26)
-    (tracks 1061)
+    (tracks 1055)
     (zones 0)
     (modules 145)
@@
     (visible_elements 7FFEFFFF)
     (pcbplotparams
-      (layerselection 0x00030_80000001)
+      (layerselection 0x010fc_80000007)
       (usegerberextensions false)
       (excludeedgelayer true)
@@
       (outputformat 1)
       (mirror false)
-      (drillshape 1)
+      (drillshape 0)
       (scaleselection 1)
-      (outputdirectory ""))
+      (outputdirectory gerber/))
   )
   (net 0 "")
@@
   (segment (start 150 82.35) (end 146.85 82.35) (width 0.2) (layer F.Cu) (net 24))
   (segment (start 146.85 82.35) (end 146.8 82.3) (width 0.2) (layer F.Cu) (net 24))
-  (segment (start 179.8 75.7) (end 179.8 75.1476) (width 0.1524) (layer F.Cu) (net 25))
-  (segment (start 162.1 56.3) (end 159.49 53.69) (width 0.1524) (layer F.Cu) (net 25))
-  (segment (start 179.8 75.1476) (end 178.5524 73.9) (width 0.1524) (layer F.Cu) (net 25))
-  (segment (start 178.5524 73.9) (end 172.8 73.9) (width 0.1524) (layer F.Cu) (net 25))
-  (segment (start 172.8 73.9) (end 169.9 71) (width 0.1524) (layer F.Cu) (net 25))
-  (segment (start 162.1 63.5) (end 162.1 56.3) (width 0.1524) (layer F.Cu) (net 25))
-  (segment (start 169.9 71) (end 169.9 66.5) (width 0.1524) (layer F.Cu) (net 25))
-  (segment (start 169.9 66.5) (end 169.1 65.7) (width 0.1524) (layer F.Cu) (net 25))
-  (segment (start 169.1 65.7) (end 164.3 65.7) (width 0.1524) (layer F.Cu) (net 25))
-  (segment (start 164.3 65.7) (end 162.1 63.5) (width 0.1524) (layer F.Cu) (net 25))
+  (segment (start 179.8 75.7) (end 175.1 75.7) (width 0.1524) (layer F.Cu) (net 25))
+  (segment (start 175.1 75.7) (end 169.9 70.5) (width 0.1524) (layer F.Cu) (net 25))
+  (segment (start 169.9 70.5) (end 169.9 64.1) (width 0.1524) (layer F.Cu) (net 25))
+  (segment (start 169.9 64.1) (end 159.49 53.69) (width 0.1524) (layer F.Cu) (net 25))
   (segment (start 159.49 53.69) (end 153.8 53.69) (width 0.1524) (layer F.Cu) (net 25))
   (segment (start 150.1 53.75) (end 150.1 52.65) (width 0.1524) (layer F.Cu) (net 25))
@@
   (segment (start 125.05 78.25) (end 125.05 79.8) (width 0.2) (layer F.Cu) (net 50))
   (segment (start 123.45 79.8) (end 125.05 79.8) (width 0.4) (layer F.Cu) (net 50))
-  (segment (start 131.45 87.9) (end 131.45 89.25) (width 0.2) (layer F.Cu) (net 51))
-  (segment (start 131.45 89.25) (end 130.6 90.1) (width 0.2) (layer F.Cu) (net 51))
-  (segment (start 130.6 90.1) (end 125.8 90.1) (width 0.2) (layer F.Cu) (net 51))
+  (segment (start 131.45 87.9) (end 130.9 87.9) (width 0.2) (layer F.Cu) (net 51))
+  (segment (start 130.9 87.9) (end 128.7 90.1) (width 0.2) (layer F.Cu) (net 51))
+  (segment (start 128.7 90.1) (end 125.8 90.1) (width 0.2) (layer F.Cu) (net 51))
   (segment (start 125.8 90.1) (end 125.05 89.35) (width 0.2) (layer F.Cu) (net 51))
   (segment (start 125.05 89.35) (end 125.05 87.8) (width 0.2) (layer F.Cu) (net 51))
@@
   (segment (start 174.3 56.9) (end 173.63 56.23) (width 0.1524) (layer F.Cu) (net 71))
   (segment (start 173.63 56.23) (end 171.8 56.23) (width 0.1524) (layer F.Cu) (net 71))
+  (segment (start 131.45 86.1) (end 130.7 86.1) (width 0.2) (layer F.Cu) (net 84))
+  (segment (start 130.7 86.1) (end 129 87.8) (width 0.2) (layer F.Cu) (net 84))
+  (segment (start 129 87.8) (end 127.95 87.8) (width 0.2) (layer F.Cu) (net 84))
   (segment (start 127.95 79.8) (end 128.9 79.8) (width 0.2) (layer F.Cu) (net 84))
   (segment (start 128.9 79.8) (end 130.2 81.1) (width 0.2) (layer F.Cu) (net 84))
@@
   (segment (start 132.2 78.4) (end 131.9 78.1) (width 0.2) (layer F.Cu) (net 84))
   (segment (start 131.9 78.1) (end 131.45 78.1) (width 0.2) (layer F.Cu) (net 84))
-  (segment (start 131.45 86.1) (end 130.8 86.1) (width 0.2) (layer F.Cu) (net 84))
-  (segment (start 130.8 86.1) (end 129.1 87.8) (width 0.2) (layer F.Cu) (net 84))
-  (segment (start 129.1 87.8) (end 127.95 87.8) (width 0.2) (layer F.Cu) (net 84))
   (segment (start 127.95 87.8) (end 127.95 83.8) (width 0.4) (layer F.Cu) (net 84))
   (segment (start 127.95 79.8) (end 127.95 83.8) (width 0.4) (layer F.Cu) (net 84))
@@
     (connect_pads (clearance 0.18))
     (min_thickness 0.18)
-    (fill yes (arc_segments 16) (thermal_gap 0.508) (thermal_bridge_width 0.508) (smoothing fillet) (radius 0.15))
+    (fill yes (arc_segments 16) (thermal_gap 0.508) (thermal_bridge_width 0.508) (smoothing fillet) (radius 0.2))
     (polygon
       (pts
@@
     (connect_pads (clearance 0.18))
     (min_thickness 0.18)
-    (fill yes (arc_segments 16) (thermal_gap 0.508) (thermal_bridge_width 0.508) (smoothing fillet) (radius 0.15))
+    (fill yes (arc_segments 16) (thermal_gap 0.508) (thermal_bridge_width 0.508) (smoothing fillet) (radius 0.2))
     (polygon
       (pts
@@
     (connect_pads (clearance 0.18))
     (min_thickness 0.18)
-    (fill yes (arc_segments 16) (thermal_gap 0.508) (thermal_bridge_width 0.508) (smoothing fillet) (radius 0.15))
+    (fill yes (arc_segments 16) (thermal_gap 0.508) (thermal_bridge_width 0.508) (smoothing fillet) (radius 0.2))
     (polygon
       (pts
@@
     (connect_pads (clearance 0.18))
     (min_thickness 0.18)
-    (fill yes (arc_segments 16) (thermal_gap 0.508) (thermal_bridge_width 0.508) (smoothing fillet) (radius 0.15))
+    (fill yes (arc_segments 16) (thermal_gap 0.508) (thermal_bridge_width 0.508) (smoothing fillet) (radius 0.2))
     (polygon
       (pts
@@
     (connect_pads (clearance 0.18))
     (min_thickness 0.18)
-    (fill yes (arc_segments 16) (thermal_gap 0.508) (thermal_bridge_width 0.508) (smoothing fillet) (radius 0.15))
+    (fill yes (arc_segments 16) (thermal_gap 0.508) (thermal_bridge_width 0.508) (smoothing fillet) (radius 0.2))
     (polygon
       (pts
@@
     (connect_pads (clearance 0.18))
     (min_thickness 0.18)
-    (fill yes (arc_segments 16) (thermal_gap 0.508) (thermal_bridge_width 0.508) (smoothing fillet) (radius 0.15))
+    (fill yes (arc_segments 16) (thermal_gap 0.508) (thermal_bridge_width 0.508) (smoothing fillet) (radius 0.2))
     (polygon
       (pts
